Commit message: Update

File: resource/tb4_raw.urdf (robot description, URDF)
Before this commit: robot turtlebot4, 48 links, 47 joints
Joints:
- joint oakd_rgb_camera_joint: origin xyz=0 0 0 rpy=0 0 0 -> xyz=0 0 0 rpy=-1.5707963267948966 0.0 -1.5707963267948966

File: resource/tb4_webots.xacro (robot description, xacro)
@@ -10,4 +10,13 @@
           <alwaysOn>true</alwaysOn>
           <updateRate>20</updateRate>
+        </ros>
+      </device>
+      <device reference="rgb_camera" type="Camera">
+        <ros>
+          <topicName>/camera/image_raw</topicName>
+          <cameraInfoTopicName>/camera/camera_info</cameraInfoTopicName>
+          <alwaysOn>true</alwaysOn>
+          <updateRate>15</updateRate>
+          <frameName>oakd_rgb_camera_optical_frame</frameName>
         </ros>
       </device>
